Commit message: removed many simulation errors with gravity and camera distortion

File: iggy_description/urdf/accessories/sick_lms1xx.urdf.xacro (robot description, xacro)
@@ -26,26 +26,58 @@
 -->
 <robot xmlns:xacro="http://ros.org/wiki/xacro">
-  <xacro:include filename="$(find iggy_description)/urdf/accessories/sick_lms1xx.urdf.xacro" />
-  <xacro:macro name="sick_lms1xx_mount" params="prefix topic">
-<turnGravityOff>false</turnGravityOff>
-    <sick_lms1xx frame="${prefix}_laser" topic="${topic}" />
-    <link name="${prefix}_laser_mount">
+  <xacro:macro name="sick_lms1xx" params="frame:=laser topic:=scan" >
+    <link name="${frame}">
+      <inertial>
+        <mass value="1.1" />
+        <origin xyz="0 0 0" />
+        <inertia ixx="${0.0833333 * 1.1 * (0.102*0.102 + 0.152*0.152)}" ixy="0.0" ixz="0.0"
+          iyy="${0.0833333 * 1.1 * (0.105*0.105 + 0.152*0.152)}" iyz="0.0"
+          izz="${0.0833333 * 1.1 * (0.105*0.105 + 0.102*0.102)}" />
+      </inertial>
       <visual>
         <origin xyz="0 0 0" rpy="0 0 0" />
         <geometry>
-          <!-- Origin of this mesh is the base of the bracket. -->
-          <mesh filename="package://iggy_description/meshes/sick-lms1xx-bracket.stl" />
+          <!-- Origin of this mesh is the focal point of the LIDAR. -->
+          <mesh filename="package://iggy_description/meshes/sick-lms1xx.dae" />
         </geometry>
-        <material name="dark_grey" />
       </visual>
+      <collision>
+        <origin xyz="0 0 -0.05" rpy="0 0 0" />
+        <geometry>
+          <box size="0.105 0.1 0.1" />
+        </geometry>
+      </collision>
     </link>
-    <joint name="${prefix}_laser_joint" type="fixed">
-      <!-- This offset is from the base of the bracket to the LIDAR's focal point. -->
-      <origin xyz="0 0 0.149" rpy="0 0 0" />
-      <parent link="${prefix}_laser_mount" />
-      <child link="${prefix}_laser" />
-    </joint>
-    <gazebo reference="${prefix}_laser_mount">
-      <material>Gazebo/DarkGrey</material>
+    <gazebo reference="${frame}">
+      <turnGravityOff>false</turnGravityOff>
+      <sensor type="ray" name="${frame}">
+        <pose>0 0 0 0 0 0</pose>
+        <visualize>false</visualize>
+        <update_rate>50</update_rate>
+        <ray>
+          <scan>
+            <horizontal>
+              <samples>720</samples>
+              <resolution>1</resolution>
+              <min_angle>-2.35619</min_angle>
+              <max_angle>2.35619</max_angle>
+            </horizontal>
+          </scan>
+          <range>
+            <min>0.10</min>
+            <max>30.0</max>
+            <resolution>0.01</resolution>
+          </range>
+          <noise>
+            <type>gaussian</type>
+            <mean>0.0</mean>
+            <stddev>0.001</stddev>
+          </noise>
+        </ray>
+        <plugin name="gazebo_ros_laser" filename="libgazebo_ros_laser.so">
+          <topicName>${topic}</topicName>
+          <frameName>${frame}</frameName>
+        </plugin>
+      </sensor>
     </gazebo>
   </xacro:macro>

File: iggy_description/urdf/depth_camera.urdf.xacro (robot description, xacro)
@@ -28,9 +28,9 @@
                     <frameName>zed_current_frame</frameName>
                     <pointCloudCutoff>1.5</pointCloudCutoff>
-                    <distortionK1>0.00000001</distortionK1>
-                    <distortionK2>0.00000001</distortionK2>
-                    <distortionK3>0.00000001</distortionK3>
-                    <distortionT1>0.00000001</distortionT1>
-                    <distortionT2>0.00000001</distortionT2>
+                    <distortionK1>0</distortionK1>
+                    <distortionK2>0</distortionK2>
+                    <distortionK3>0</distortionK3>
+                    <distortionT1>0</distortionT1>
+                    <distortionT2>0</distortionT2>
                     <linesOnly>1</linesOnly>
                 </plugin>
