Commit message: improved iggy sim model

File: iggy_description/urdf/accessories/camera_mount.urdf.xacro (robot description, xacro)
@@ -1,2 +1,3 @@
+<?xml version="1.0"?>
 <robot xmlns:xacro="http://ros.org/wiki/xacro">
   <xacro:macro name="camera_mount" params="prefix tilt:=0">

File: iggy_description/urdf/depth_camera.urdf.xacro (robot description, xacro)
@@ -15,5 +15,5 @@
                     <clip>
                         <near>0.01</near>
-                        <far>5</far>
+                        <far>25</far>
                     </clip>
                 </camera>
@@ -39,5 +39,6 @@
         <link name="left_camera">
             <visual>
-                <origin xyz="0 0 0" rpy="0 1.57 0" />
+                <!-- <origin xyz="0 0 0" rpy="0 1.57 0" /> -->
+                <origin xyz="0 0 0" rpy="0 0 0" />
                 <geometry>
                     <cylinder radius="0.007" length=".031" />
@@ -50,5 +51,6 @@
         <link name="right_camera">
             <visual>
-                <origin xyz="0 0 0" rpy="0 1.57 0" />
+                <!-- <origin xyz="0 0 0" rpy="0 1.57 0" /> -->
+                <origin xyz="0 0 0" rpy="0 0 0" />
                 <geometry>
                     <cylinder radius="0.007" length=".031" />
@@ -70,4 +72,5 @@
             </visual>
         </link>
+<!--
         <link name="camera_arm">
             <visual>
@@ -80,5 +83,5 @@
                 </material>
             </visual>
-        </link>
+        </link> -->
         <joint name="left_camera_joint" type="fixed">
             <parent link="camera_center" />
@@ -96,7 +99,8 @@
             <parent link="camera_center" />
             <child link="zed_current_frame" />
-            <origin rpy="-1.57 0 -1.57" xyz="0 0 0" />
+            <origin rpy="0 0 0" xyz="0 0 0" />
+            <!-- <origin rpy="-1.57 0 -1.57" xyz="0 0 0" /> -->
         </joint>
-        <joint name="camera_center_joint" type="fixed">
+<!--        <joint name="camera_center_joint" type="fixed">
             <parent link="camera_arm" />
             <child link="camera_center" />
@@ -107,5 +111,5 @@
             <child link="camera_arm" />
             <origin rpy="0 0 0" xyz="0 0 0.25" />
-        </joint>
+        </joint> -->
     </xacro:macro>
 </robot>

File: iggy_description/urdf/iggy2.urdf.xacro (robot description, xacro)
@@ -257,4 +257,13 @@
         <material>Gazebo/Orange</material>
     </gazebo>
+  <xacro:include filename="depth_camera.urdf.xacro" />
+  <xacro:depth_camera>
+    <origin xyz="0 0 0" rpy="0 0 0" />
+  </xacro:depth_camera>
+    <joint name="base_link_to_camera" type="fixed">
+        <parent link="base_link" />
+        <child link="camera_center" />
+        <origin xyz="0.125 0 1.1" rpy="0 0.785398 0" />
+    </joint>
 <!--Plugins -->
     <gazebo>
