Commit message: implemented depth camera

File: iggy_description/urdf/depth_camera.urdf.xacro (robot description, xacro)
@@ -2,31 +2,107 @@
 <robot xmlns:xacro="http://ros.org/wiki/xacro">
     <xacro:macro name="depth_camera">
-        <link name="depth_camera_link">
-            <visual>
-                <origin xyz="0 0 0" rpy="0 1.57 0"/>
-                <geometry>
-                    <cylinder radius="0.017" length=".031"/>
-                </geometry>
-                <material name="dark_grey">
-                    <color rgba="0.1 0.1 0.1 1"/>
-                </material>
-            </visual>
-     <sensor type="depth" name="depth_camera">
-        <always_on>true</always_on>
-        <update_rate>20.0</update_rate>
-        <camera>
-          <horizontal_fov>${57.0*3.141/180.0}</horizontal_fov>
-          <image>
-            <format>B8G8R8</format>
-            <width>640</width>
-            <height>480</height>
-          </image>
-          <clip>
-            <near>0.01</near>
-            <far>5</far>
-          </clip>
-        </camera>
-      </sensor>
-        </link>
-  </xacro:macro>
+        <gazebo reference="camera_center">
+            <sensor type="depth" name="depth_camera">
+                <always_on>true</always_on>
+                <update_rate>20.0</update_rate>
+                <camera>
+                    <horizontal_fov>${57.0*3.141/180.0}</horizontal_fov>
+                    <image>
+                        <format>B8G8R8</format>
+                        <width>640</width>
+                        <height>480</height>
+                    </image>
+                    <clip>
+                        <near>0.01</near>
+                        <far>5</far>
+                    </clip>
+                </camera>
+                <plugin name="depth_camera_frame_controller" filename="libgazebo_ros_depth_camera.so">
+                    <always_on>true</always_on>
+                    <updateRate>20.0</updateRate>
+                    <cameraName>depth_camera</cameraName>
+                    <imageTopicName>rgb/image_raw</imageTopicName>
+                    <pointCloudTopicName>rgb/points</pointCloudTopicName>
+                    <cameraInfoTopicName>rgb/camera_info</cameraInfoTopicName>
+                    <frameName>depth_camera_optical</frameName>
+                    <pointCloudCutoff>1.5</pointCloudCutoff>
+                    <distortionK1>0.00000001</distortionK1>
+                    <distortionK2>0.00000001</distortionK2>
+                    <distortionK3>0.00000001</distortionK3>
+                    <distortionT1>0.00000001</distortionT1>
+                    <distortionT2>0.00000001</distortionT2>
+                </plugin>
+            </sensor>
+        </gazebo>
+   <link name="left_camera">
+        <visual>
+            <origin xyz="0 0 0" rpy="0 1.57 0"/>
+            <geometry>
+                <cylinder radius="0.007" length=".031"/>
+            </geometry>
+            <material name="dark_grey">
+                <color rgba="0.1 0.1 0.1 1"/>
+            </material>
+        </visual>
+    </link>
+    <link name="camera_center">
+        <visual>
+            <origin xyz="0 0 0" rpy="0 0 0"/>
+            <geometry>
+                <mesh filename="package://iggy_description/meshes/zed.stl" />
+            </geometry>
+            <material name="light_grey">
+                <color rgba="0.8 0.8 0.8 0.8"/>
+            </material>
+        </visual>
+    </link>
+    <link name="camera_arm">
+        <visual>
+            <origin xyz="0 0 0" rpy="0 0 0"/>
+            <geometry>
+                <cylinder radius="0.007" length=".51"/>
+            </geometry>
+            <material name="dark_grey">
+                <color rgba="0.1 0.1 0.1 1"/>
+            </material>
+        </visual>
+    </link>
+    <link name="right_camera">
+        <visual>
+            <origin xyz="0 0 0" rpy="0 1.57 0"/>
+            <geometry>
+                <cylinder radius="0.007" length=".031"/>
+            </geometry>
+            <material name="dark_grey">
+                <color rgba="0.1 0.1 0.1 1"/>
+            </material>
+        </visual>
+    </link>
+    <joint name="left_camera_joint" type="fixed">
+        <parent link="camera_center"/>
+        <child link="left_camera"/>
+        <origin xyz="0 0.06 0" rpy="0 0 0" />
+    </joint>
+    <joint name="right_camera_joint" type="fixed">
+        <parent link="camera_center"/>
+        <child link="right_camera"/>
+        <origin xyz="0 -0.06 0" rpy="0 0 0" />
+    </joint>
+  <link name="depth_camera_optical"></link>
+    <joint name="depth_camera_optical_joint" type="fixed">
+      <parent link="camera_center"/>
+      <child link="depth_camera_optical"/>
+      <origin rpy="-1.57 0 -1.57" xyz="0 0 0"/>
+    </joint>
+    <joint name="camera_arm_joint" type="fixed">
+      <parent link="mid_mount"/>
+      <child link="camera_arm"/>
+      <origin rpy="0 0 0" xyz="0 0 0"/>
+    </joint>
+    <joint name="camera_center_joint" type="fixed">
+      <parent link="camera_arm"/>
+      <child link="camera_center"/>
+      <origin rpy="0 0.24 0" xyz="0 0 0.25"/>
+    </joint>
+    </xacro:macro>
 </robot>

File: iggy_description/urdf/iggy.urdf.xacro (robot description, xacro)
@@ -174,19 +174,12 @@
   <!-- Optional custom includes. -->
   <xacro:include filename="$(optenv IGGY_URDF_EXTRAS empty.urdf)" />
-  <!--
-  <joint name="zed_left_camera_joint" type="fixed">
+ <!--
+  <link name="depth_camera_mount"></link>
+  <joint name="depth_camera_mount" type="fixed">
     <parent link="front_mount" />
-    <child link="zed_left_camera" />
-    <origin xyz="${mount_spacing} 0.06 0" />
-  </joint>
-  <xacro:include filename="zed_camera.urdf.xacro" />
-  <xacro:zed_camera prefix="zed_camera"/>
+    <child link="depth_camera_mount" />
+    <origin xyz="${mount_spacing} 0.00 0.20" />
+  </joint>   -->
   <xacro:include filename="depth_camera.urdf.xacro" />
   <xacro:depth_camera/>
-  <joint name="depth_camera_joint" type="fixed">
-    <parent link="front_mount" />
-    <child link="depth_camera_link" />
-    <origin xyz="${mount_spacing} 0.06 0" />
-  </joint>
- -->
 </robot>

Commit message: white line detection works in simualtion. still need to integrate pointcloud

File: iggy_description/urdf/depth_camera.urdf.xacro (robot description, xacro)
@@ -18,5 +18,5 @@
                     </clip>
                 </camera>
-                <plugin name="depth_camera_frame_controller" filename="libgazebo_ros_depth_camera.so">
+                <plugin name="depth_camera_frame_controller" filename="libgazebo_tutorials.so">
                     <always_on>true</always_on>
                     <updateRate>20.0</updateRate>
@@ -35,74 +35,75 @@
             </sensor>
         </gazebo>
-   <link name="left_camera">
-        <visual>
-            <origin xyz="0 0 0" rpy="0 1.57 0"/>
-            <geometry>
-                <cylinder radius="0.007" length=".031"/>
-            </geometry>
-            <material name="dark_grey">
-                <color rgba="0.1 0.1 0.1 1"/>
-            </material>
-        </visual>
-    </link>
-    <link name="camera_center">
-        <visual>
-            <origin xyz="0 0 0" rpy="0 0 0"/>
-            <geometry>
-                <mesh filename="package://iggy_description/meshes/zed.stl" />
-            </geometry>
-            <material name="light_grey">
-                <color rgba="0.8 0.8 0.8 0.8"/>
-            </material>
-        </visual>
-    </link>
-    <link name="camera_arm">
-        <visual>
-            <origin xyz="0 0 0" rpy="0 0 0"/>
-            <geometry>
-                <cylinder radius="0.007" length=".51"/>
-            </geometry>
-            <material name="dark_grey">
-                <color rgba="0.1 0.1 0.1 1"/>
-            </material>
-        </visual>
-    </link>
-    <link name="right_camera">
-        <visual>
-            <origin xyz="0 0 0" rpy="0 1.57 0"/>
-            <geometry>
-                <cylinder radius="0.007" length=".031"/>
-            </geometry>
-            <material name="dark_grey">
-                <color rgba="0.1 0.1 0.1 1"/>
-            </material>
-        </visual>
-    </link>
-    <joint name="left_camera_joint" type="fixed">
-        <parent link="camera_center"/>
-        <child link="left_camera"/>
-        <origin xyz="0 0.06 0" rpy="0 0 0" />
-    </joint>
-    <joint name="right_camera_joint" type="fixed">
-        <parent link="camera_center"/>
-        <child link="right_camera"/>
-        <origin xyz="0 -0.06 0" rpy="0 0 0" />
-    </joint>
-  <link name="depth_camera_optical"></link>
-    <joint name="depth_camera_optical_joint" type="fixed">
-      <parent link="camera_center"/>
-      <child link="depth_camera_optical"/>
-      <origin rpy="-1.57 0 -1.57" xyz="0 0 0"/>
-    </joint>
-    <joint name="camera_arm_joint" type="fixed">
-      <parent link="mid_mount"/>
-      <child link="camera_arm"/>
-      <origin rpy="0 0 0" xyz="0 0 0"/>
-    </joint>
-    <joint name="camera_center_joint" type="fixed">
-      <parent link="camera_arm"/>
-      <child link="camera_center"/>
-      <origin rpy="0 0.24 0" xyz="0 0 0.25"/>
-    </joint>
+        <link name="left_camera">
+            <visual>
+                <origin xyz="0 0 0" rpy="0 1.57 0" />
+                <geometry>
+                    <cylinder radius="0.007" length=".031" />
+                </geometry>
+                <material name="dark_grey">
+                    <color rgba="0.1 0.1 0.1 1" />
+                </material>
+            </visual>
+        </link>
+        <link name="right_camera">
+            <visual>
+                <origin xyz="0 0 0" rpy="0 1.57 0" />
+                <geometry>
+                    <cylinder radius="0.007" length=".031" />
+                </geometry>
+                <material name="dark_grey">
+                    <color rgba="0.1 0.1 0.1 1" />
+                </material>
+            </visual>
+        </link>
+        <link name="camera_center">
+            <visual>
+                <origin xyz="0 0 0" rpy="0 0 0" />
+                <geometry>
+                    <mesh filename="package://iggy_description/meshes/zed.stl" />
+                </geometry>
+                <material name="light_grey">
+                    <color rgba="0.8 0.8 0.8 0.8" />
+                </material>
+            </visual>
+        </link>
+        <link name="camera_arm">
+            <visual>
+                <origin xyz="0 0 0" rpy="0 0 0" />
+                <geometry>
+                    <cylinder radius="0.007" length=".50" />
+                </geometry>
+                <material name="dark_grey">
+                    <color rgba="0.1 0.1 0.1 1" />
+                </material>
+            </visual>
+        </link>
+        <joint name="left_camera_joint" type="fixed">
+            <parent link="camera_center" />
+            <child link="left_camera" />
+            <origin xyz="0 0.06 0" rpy="0 0 0" />
+        </joint>
+        <joint name="right_camera_joint" type="fixed">
+            <parent link="camera_center" />
+            <child link="right_camera" />
+            <origin xyz="0 -0.06 0" rpy="0 0 0" />
+        </joint>
+        <!-- Align the optical frame to the camera frame -->
+        <link name="depth_camera_optical"></link>
+        <joint name="depth_camera_optical_joint" type="fixed">
+            <parent link="camera_center" />
+            <child link="depth_camera_optical" />
+            <origin rpy="-1.57 0 -1.57" xyz="0 0 0" />
+        </joint>
+        <joint name="camera_center_joint" type="fixed">
+            <parent link="camera_arm" />
+            <child link="camera_center" />
+            <origin rpy="0 0 0" xyz="0 0 0.25" />
+        </joint>
+        <joint name="camera_arm_joint" type="fixed">
+            <parent link="mid_mount" />
+            <child link="camera_arm" />
+            <origin rpy="0 0 0" xyz="0 0 0" />
+        </joint>
     </xacro:macro>
 </robot>

File: iggy_description/urdf/iggy.urdf.xacro (robot description, xacro)
@@ -182,4 +182,6 @@
   </joint>   -->
   <xacro:include filename="depth_camera.urdf.xacro" />
-  <xacro:depth_camera/>
+  <xacro:depth_camera>
+    <origin xyz="0 0 ${chassis_height}" rpy="0 0 0" />
+  </xacro:depth_camera>
 </robot>

Commit message: some sucess with vision to cost map. FIX points appear below the map

File: iggy_description/urdf/depth_camera.urdf.xacro (robot description, xacro)
@@ -24,7 +24,7 @@
                     <cameraName>depth_camera</cameraName>
                     <imageTopicName>rgb/image_raw</imageTopicName>
-                    <pointCloudTopicName>rgb/points</pointCloudTopicName>
+                    <pointCloudTopicName>/point_cloud/white_cloud</pointCloudTopicName>
                     <cameraInfoTopicName>rgb/camera_info</cameraInfoTopicName>
-                    <frameName>depth_camera_optical</frameName>
+                    <frameName>zed_current_frame</frameName>
                     <pointCloudCutoff>1.5</pointCloudCutoff>
                     <distortionK1>0.00000001</distortionK1>
@@ -92,8 +92,8 @@
         </joint>
         <!-- Align the optical frame to the camera frame -->
-        <link name="depth_camera_optical"></link>
-        <joint name="depth_camera_optical_joint" type="fixed">
+        <link name="zed_current_frame"></link>
+        <joint name="zed_current_frame_joint" type="fixed">
             <parent link="camera_center" />
-            <child link="depth_camera_optical" />
+            <child link="zed_current_frame" />
             <origin rpy="-1.57 0 -1.57" xyz="0 0 0" />
         </joint>

File: iggy_description/urdf/iggy.urdf.xacro (robot description, xacro)
@@ -97,5 +97,5 @@
       <!-- Center of mass -->
       <origin xyz="0.012  0.002 0.067" rpy="0 0 0"/>
-      <mass value="16.523"/>
+      <mass value="86.523"/>
       <!-- Moments of inertia: ( chassis without wheels ) -->
       <inertia
@@ -170,15 +170,8 @@
   <!-- Optional standard accessories, including their simulation data. The rendering
        of these into the final description is controlled by optenv variables, which
-       default each one to off.-->
+       default each one to off.  -->
   <xacro:include filename="accessories.urdf.xacro" />
   <!-- Optional custom includes. -->
   <xacro:include filename="$(optenv IGGY_URDF_EXTRAS empty.urdf)" />
- <!--
-  <link name="depth_camera_mount"></link>
-  <joint name="depth_camera_mount" type="fixed">
-    <parent link="front_mount" />
-    <child link="depth_camera_mount" />
-    <origin xyz="${mount_spacing} 0.00 0.20" />
-  </joint>   -->
   <xacro:include filename="depth_camera.urdf.xacro" />
   <xacro:depth_camera>

Commit message: removed unneeded igvc_2dnav, moved the camera up and angled down, increase speed of robot

File: iggy_description/urdf/depth_camera.urdf.xacro (robot description, xacro)
@@ -7,5 +7,5 @@
                 <update_rate>20.0</update_rate>
                 <camera>
-                    <horizontal_fov>${57.0*3.141/180.0}</horizontal_fov>
+                    <horizontal_fov>${110.0*3.141/180.0}</horizontal_fov>
                     <image>
                         <format>B8G8R8</format>
@@ -101,10 +101,10 @@
             <parent link="camera_arm" />
             <child link="camera_center" />
-            <origin rpy="0 0 0" xyz="0 0 0.25" />
+            <origin rpy="0 0.30 0" xyz="0 0 0.25" />
         </joint>
         <joint name="camera_arm_joint" type="fixed">
             <parent link="mid_mount" />
             <child link="camera_arm" />
-            <origin rpy="0 0 0" xyz="0 0 0" />
+            <origin rpy="0 0 0" xyz="0 0 0.25" />
         </joint>
     </xacro:macro>

File: iggy_description/urdf/iggy.urdf.xacro (robot description, xacro)
@@ -96,5 +96,5 @@
     <inertial>
       <!-- Center of mass -->
-      <origin xyz="0.012  0.002 0.067" rpy="0 0 0"/>
+      <origin xyz="0.012  0.002 0.007" rpy="0 0 0"/>
       <mass value="86.523"/>
       <!-- Moments of inertia: ( chassis without wheels ) -->

Commit message: converging sim and irl

File: iggy_description/urdf/depth_camera.urdf.xacro (robot description, xacro)
@@ -7,5 +7,5 @@
                 <update_rate>20.0</update_rate>
                 <camera>
-                    <horizontal_fov>${57.0*3.141/180.0}</horizontal_fov>
+                    <horizontal_fov>${110.0*3.141/180.0}</horizontal_fov>
                     <image>
                         <format>B8G8R8</format>
@@ -18,18 +18,20 @@
                     </clip>
                 </camera>
-                <plugin name="depth_camera_frame_controller" filename="libgazebo_tutorials.so">
+                 <plugin name="depth_camera_frame_controller" filename="libgazebo_iggy_vision.so">
+                <!-- <plugin name="depth_camera_frame_controller" filename="libgazebo_ros_depth_camera.so"> -->
                     <always_on>true</always_on>
                     <updateRate>20.0</updateRate>
                     <cameraName>depth_camera</cameraName>
                     <imageTopicName>rgb/image_raw</imageTopicName>
-                    <pointCloudTopicName>rgb/points</pointCloudTopicName>
+                    <pointCloudTopicName>/point_cloud/white_cloud</pointCloudTopicName>
                     <cameraInfoTopicName>rgb/camera_info</cameraInfoTopicName>
-                    <frameName>depth_camera_optical</frameName>
+                    <frameName>zed_current_frame</frameName>
                     <pointCloudCutoff>1.5</pointCloudCutoff>
-                    <distortionK1>0.00000001</distortionK1>
-                    <distortionK2>0.00000001</distortionK2>
-                    <distortionK3>0.00000001</distortionK3>
-                    <distortionT1>0.00000001</distortionT1>
-                    <distortionT2>0.00000001</distortionT2>
+                    <distortionK1>0</distortionK1>
+                    <distortionK2>0</distortionK2>
+                    <distortionK3>0</distortionK3>
+                    <distortionT1>0</distortionT1>
+                    <distortionT2>0</distortionT2>
+                    <linesOnly>1</linesOnly>
                 </plugin>
             </sensor>
@@ -90,8 +92,8 @@
         </joint>
         <!-- Align the optical frame to the camera frame -->
-        <link name="depth_camera_optical"></link>
-        <joint name="depth_camera_optical_joint" type="fixed">
+        <link name="zed_current_frame"></link>
+        <joint name="zed_current_frame_joint" type="fixed">
             <parent link="camera_center" />
-            <child link="depth_camera_optical" />
+            <child link="zed_current_frame" />
             <origin rpy="-1.57 0 -1.57" xyz="0 0 0" />
         </joint>
@@ -99,10 +101,10 @@
             <parent link="camera_arm" />
             <child link="camera_center" />
-            <origin rpy="0 0 0" xyz="0 0 0.25" />
+            <origin rpy="0 0.30 0" xyz="0 0 0.25" />
         </joint>
         <joint name="camera_arm_joint" type="fixed">
             <parent link="mid_mount" />
             <child link="camera_arm" />
-            <origin rpy="0 0 0" xyz="0 0 0" />
+            <origin rpy="0 0 0" xyz="0 0 0.25" />
         </joint>
     </xacro:macro>

File: iggy_description/urdf/iggy.urdf.xacro (robot description, xacro)
@@ -96,6 +96,6 @@
     <inertial>
       <!-- Center of mass -->
-      <origin xyz="0.012  0.002 0.067" rpy="0 0 0"/>
-      <mass value="16.523"/>
+      <origin xyz="0.012  0.002 0.007" rpy="0 0 0"/>
+      <mass value="86.523"/>
       <!-- Moments of inertia: ( chassis without wheels ) -->
       <inertia
@@ -170,15 +170,8 @@
   <!-- Optional standard accessories, including their simulation data. The rendering
        of these into the final description is controlled by optenv variables, which
-       default each one to off.-->
+       default each one to off.  -->
   <xacro:include filename="accessories.urdf.xacro" />
   <!-- Optional custom includes. -->
   <xacro:include filename="$(optenv IGGY_URDF_EXTRAS empty.urdf)" />
- <!--
-  <link name="depth_camera_mount"></link>
-  <joint name="depth_camera_mount" type="fixed">
-    <parent link="front_mount" />
-    <child link="depth_camera_mount" />
-    <origin xyz="${mount_spacing} 0.00 0.20" />
-  </joint>   -->
   <xacro:include filename="depth_camera.urdf.xacro" />
   <xacro:depth_camera>
