Commit message: adjusted iggy urdf to be level

File: iggy_description/urdf/iggy2.urdf (robot description, URDF)
Before this commit: robot iggy, 9 links, 8 joints
Links:
- link front_wheel_base: geometry collision box size=0.11 0.60 0.25; visual box size=0.11 0.60 0.25
Joints:
- joint cfl_pivot_joint: origin xyz=0 0.15 -0.1475 rpy=0 0 0 -> xyz=0 0.21 -0.147 rpy=0 0 0
- joint cfr_pivot_joint: origin xyz=0 -0.15 -0.1475 rpy=0 0 0 -> xyz=0 -0.21 -0.1475 rpy=0 0 0
- joint front_left_wheel_joint: origin xyz=-0.03 0 -0.0925 rpy=0 0 0 -> xyz=-0.03 0 -0.093 rpy=0 0 0
- joint front_wheel_base_to_base_link: origin xyz=0.38 0 -0.275 rpy=0 0 0 -> xyz=0.38 0 -0.265 rpy=0 0 0
