Commit message: added zed to robot still need to add zed driver

File: iggy_description/urdf/iggy.urdf.xacro (robot description, xacro)
@@ -174,3 +174,10 @@
   <!-- Optional custom includes. -->
   <xacro:include filename="$(optenv IGGY_URDF_EXTRAS empty.urdf)" />
+  <joint name="zed_left_camera_joint" type="fixed">
+    <parent link="front_mount" />
+    <child link="zed_left_camera" />
+    <origin xyz="${mount_spacing} 0 0" />
+  </joint>
+  <xacro:include filename="zed_camera.urdf.xacro" />
+  <xacro:zed_camera prefix="zed_camera"/>
 </robot>

Commit message: with two cameras and move base working, no stereo vision, and move basee needs tunning

File: iggy_description/urdf/iggy.urdf.xacro (robot description, xacro)
@@ -174,10 +174,19 @@
   <!-- Optional custom includes. -->
   <xacro:include filename="$(optenv IGGY_URDF_EXTRAS empty.urdf)" />
+  <!--
   <joint name="zed_left_camera_joint" type="fixed">
     <parent link="front_mount" />
     <child link="zed_left_camera" />
-    <origin xyz="${mount_spacing} 0 0" />
+    <origin xyz="${mount_spacing} 0.06 0" />
   </joint>
   <xacro:include filename="zed_camera.urdf.xacro" />
   <xacro:zed_camera prefix="zed_camera"/>
+  <xacro:include filename="depth_camera.urdf.xacro" />
+  <xacro:depth_camera/>
+  <joint name="depth_camera_joint" type="fixed">
+    <parent link="front_mount" />
+    <child link="depth_camera_link" />
+    <origin xyz="${mount_spacing} 0.06 0" />
+  </joint>
+ -->
 </robot>

Commit message: cleaning up the goal_pub_IGVC.py code to make it work better as per code-review with MAJ Larkin. Also fixed simulation turning urdf paramter.

File: iggy_description/urdf/iggy.urdf.xacro (robot description, xacro)
@@ -97,6 +97,6 @@
       <!-- Center of mass -->
       <origin xyz="0.012  0.002 0.067" rpy="0 0 0"/>
-      <mass value="86.523"/>
-      <!-- Moments of inertia: ( chassis without wheels ) -->
+      <mass value="16.523"/>
+      <!-- Moments of inertia: ( chassis without wheels ) changing the mass value here to a higher one will mess up turning -->
       <inertia
         ixx="0.3136" ixy="-0.0008" ixz="0.0164"
