Commit message: modified iggy.urdf.xacro to work again but is now moving backwards. Fixed waypoint publisher.

File: iggy_description/urdf/accessories.urdf.xacro (robot description, xacro)
@@ -17,5 +17,5 @@
   <xacro:if value="$(optenv IGGY_LASER 0)">
     <sick_lms1xx_mount prefix="$(optenv IGGY_LASER_MOUNT front)"
-                       topic="$(optenv IGGY_LASER_TOPIC front/scan)"/>
+                       topic="$(optenv IGGY_LASER_TOPIC /scan)"/>
     <joint name="$(optenv IGGY_LASER_MOUNT front)_laser_mount_joint" type="fixed">
       <origin xyz="$(optenv IGGY_LASER_OFFSET 0 0 0)"

File: iggy_description/urdf/depth_camera.urdf.xacro (robot description, xacro)
@@ -72,16 +72,4 @@
             </visual>
         </link>
-<!--
-        <link name="camera_arm">
-            <visual>
-                <origin xyz="0 0 0" rpy="0 0 0" />
-                <geometry>
-                    <cylinder radius="0.007" length=".50" />
-                </geometry>
-                <material name="dark_grey">
-                    <color rgba="0.1 0.1 0.1 1" />
-                </material>
-            </visual>
-        </link> -->
         <joint name="left_camera_joint" type="fixed">
             <parent link="camera_center" />
@@ -102,14 +90,4 @@
             <!-- <origin rpy="-1.57 0 -1.57" xyz="0 0 0" /> -->
         </joint>
-<!--        <joint name="camera_center_joint" type="fixed">
-            <parent link="camera_arm" />
-            <child link="camera_center" />
-            <origin rpy="0 0.30 0" xyz="0 0 0.25" />
-        </joint>
-        <joint name="camera_arm_joint" type="fixed">
-            <parent link="mid_mount" />
-            <child link="camera_arm" />
-            <origin rpy="0 0 0" xyz="0 0 0.25" />
-        </joint> -->
     </xacro:macro>
 </robot>

File: iggy_description/urdf/iggy.urdf.xacro (robot description, xacro)
@@ -178,3 +178,24 @@
     <origin xyz="0 0 ${chassis_height}" rpy="0 0 0" />
   </xacro:depth_camera>
+        <link name="camera_arm">
+            <visual>
+                <origin xyz="0 0 0" rpy="0 0 0" />
+                <geometry>
+                    <cylinder radius="0.007" length=".50" />
+                </geometry>
+                <material name="dark_grey">
+                    <color rgba="0.1 0.1 0.1 1" />
+                </material>
+            </visual>
+        </link>
+        <joint name="camera_center_joint" type="fixed">
+            <parent link="camera_arm" />
+            <child link="camera_center" />
+            <origin rpy="0 0.30 0" xyz="0 0 0.25" />
+        </joint>
+        <joint name="camera_arm_joint" type="fixed">
+            <parent link="mid_mount" />
+            <child link="camera_arm" />
+            <origin rpy="0 0 0" xyz="0 0 0.25" />
+        </joint>
 </robot>
